Commit message: fix crash-prone prim paths and URDF mesh URIs; add fork notes
- Move L/R observation prim paths out of param_config into task/scene_prims.py,
  pointing at task_board_color (snap anchor) instead of rod_16mm (snap child)
  to prevent PhysX tensor-view crashes mid-sequence.
- Rewrite all 90 URDF mesh filenames from absolute file:///Yejun_Files/...
  paths to relative meshes/<file>.obj so the URDF resolves on any machine.
- Add README_FORK.md: use play2perfect/.venv_isaacsim (isaacsim 5.1.0.0)
  instead of uv sync; document the two fixes above.

File: robot/vega_1u_gripper.urdf (robot description, URDF)
Before this commit: robot vega_1u_gripper, 35 links, 34 joints
Links:
- link L_arm_l2: geometry collision mesh filename=meshes/L_arm_l2_collisions_arm_l2_mesh.obj scale=1. 1. 1.; visual mesh filename=meshes/L_arm_l2_collisions_arm_l2_mesh.obj scale=1. 1. 1.
- link L_arm_l3: geometry collision mesh filename=meshes/L_arm_l3_collisions_arm_l3_mesh.obj scale=1. 1. 1.; visual mesh filename=meshes/L_arm_l3_collisions_arm_l3_mesh.obj scale=1. 1. 1.
- link L_arm_l4: geometry collision mesh filename=meshes/L_arm_l4_collisions_arm_l4_mesh.obj scale=1. 1. 1.; visual mesh filename=meshes/L_arm_l4_collisions_arm_l4_mesh.obj scale=1. 1. 1.
- link L_arm_l5: geometry collision mesh filename=meshes/L_arm_l5_collisions_arm_l5_mesh.obj scale=1. 1. 1.; visual mesh filename=meshes/L_arm_l5_collisions_arm_l5_mesh.obj scale=1. 1. 1.
- link L_arm_l7: geometry collision mesh filename=meshes/L_arm_l7_collisions_arm_l7_0_mesh.obj scale=1. 1. 1.; collision mesh filename=meshes/L_arm_l7_collisions_arm_l7_1_mesh.obj scale=1. 1. 1.
- link L_arm_l8: geometry collision mesh filename=meshes/L_arm_l8_collisions_arm_l8_mesh.obj scale=1. 1. 1.; visual mesh filename=meshes/L_arm_l8_collisions_arm_l8_mesh.obj scale=1. 1. 1.
- link L_ee_link_gripper_active_link: geometry collision mesh filename=meshes/L_ee_link_gripper_active_link_gripper_active_link.obj scale=1. 1. 1.; visual mesh filename=meshes/L_ee_link_gripper_active_link_gripper_active_link.obj scale=1. 1. 1.
- link L_ee_link_gripper_link: geometry collision mesh filename=meshes/L_ee_link_gripper_link_gripper_link.obj scale=1. 1. 1.; visual mesh filename=meshes/L_ee_link_gripper_link_gripper_ee_link_gripper_ee_li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 scale=1. 1. 1.
- link L_ee_link_gripper_passive_link: geometry collision mesh filename=meshes/L_ee_link_gripper_passive_link_left_gripper_passive_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 scale=1. 1. 1.; visual mesh filename=meshes/L_ee_link_gripper_passive_link_left_gripper_passive_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 scale=1. 1. 1.
- link R_arm_l2: geometry collision mesh filename=meshes/R_arm_l2_collisions_arm_l2_mesh.obj scale=1. 1. 1.; visual mesh filename=meshes/R_arm_l2_collisions_arm_l2_mesh.obj scale=1. 1. 1.
- link R_arm_l3: geometry collision mesh filename=meshes/R_arm_l3_collisions_arm_l3_mesh.obj scale=1. 1. 1.; visual mesh filename=meshes/R_arm_l3_collisions_arm_l3_mesh.obj scale=1. 1. 1.
- link R_arm_l4: geometry collision mesh filename=meshes/R_arm_l4_collisions_arm_l4_mesh.obj scale=1. 1. 1.; visual mesh filename=meshes/R_arm_l4_collisions_arm_l4_mesh.obj scale=1. 1. 1.
- link R_arm_l5: geometry collision mesh filename=meshes/R_arm_l5_collisions_arm_l5_mesh.obj scale=1. 1. 1.; visual mesh filename=meshes/R_arm_l5_collisions_arm_l5_mesh.obj scale=1. 1. 1.
- link R_arm_l7: geometry collision mesh filename=meshes/R_arm_l7_collisions_arm_l7_0_mesh.obj scale=1. 1. 1.; collision mesh filename=meshes/R_arm_l7_collisions_arm_l7_1_mesh.obj scale=1. 1. 1.
- link R_arm_l8: geometry collision mesh filename=meshes/R_arm_l8_collisions_arm_l8_mesh.obj scale=1. 1. 1.; visual mesh filename=meshes/R_arm_l8_collisions_arm_l8_mesh.obj scale=1. 1. 1.
- link R_ee_link_gripper_active_link: geometry collision mesh filename=meshes/R_ee_link_gripper_active_link_gripper_active_link.obj scale=1. 1. 1.; visual mesh filename=meshes/R_ee_link_gripper_active_link_gripper_active_link.obj scale=1. 1. 1.
- link R_ee_link_gripper_link: geometry collision mesh filename=meshes/R_ee_link_gripper_link_gripper_link.obj scale=1. 1. 1.; visual mesh filename=meshes/R_ee_link_gripper_link_gripper_ee_link_gripper_ee_li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 scale=1. 1. 1.
- link R_ee_link_gripper_passive_link: geometry collision mesh filename=meshes/R_ee_link_gripper_passive_link_left_gripper_passive_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 scale=1. 1. 1.; visual mesh filename=meshes/R_ee_link_gripper_passive_link_left_gripper_passive_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 scale=1. 1. 1.
- link torso_flip_link: geometry collision mesh filename=meshes/torso_flip_link_collisions_torso_link_mesh.obj scale=1. 1. 1.; visual mesh filename=meshes/torso_flip_link_collisions_torso_link_mesh.obj scale=1. 1. 1.
- link vega_1u_L_arm_l1: geometry collision mesh filename=meshes/vega_1u_L_arm_l1_collisions_L_arm_l1_mesh.obj scale=1. 1. 1.; visual mesh filename=meshes/vega_1u_L_arm_l1_collisions_L_arm_l1_mesh.obj scale=1. 1. 1.
- link vega_1u_L_arm_l6: geometry collision mesh filename=meshes/vega_1u_L_arm_l6_collisions_L_arm_l6_mesh.obj scale=1. 1. 1.; visual mesh filename=meshes/vega_1u_L_arm_l6_collisions_L_arm_l6_mesh.obj scale=1. 1. 1.
- link vega_1u_R_arm_l1: geometry collision mesh filename=meshes/vega_1u_R_arm_l1_collisions_R_arm_l1_mesh.obj scale=1. 1. 1.; visual mesh filename=meshes/vega_1u_R_arm_l1_collisions_R_arm_l1_mesh.obj scale=1. 1. 1.
- link vega_1u_R_arm_l6: geometry collision mesh filename=meshes/vega_1u_R_arm_l6_collisions_R_arm_l6_mesh.obj scale=1. 1. 1.; visual mesh filename=meshes/vega_1u_R_arm_l6_collisions_R_arm_l6_mesh.obj scale=1. 1. 1.
- link vega_1u_base_link: geometry collision mesh filename=meshes/vega_1u_base_link_collisions_base_link_mesh.obj scale=1. 1. 1.; visual mesh filename=meshes/vega_1u_base_link_collisions_base_link_mesh.obj scale=1. 1. 1.
- link vega_1u_head_l1: geometry collision mesh filename=meshes/head_l1_0_mesh.obj scale=1. 1. 1.; collision mesh filename=meshes/head_l1_1_mesh.obj scale=1. 1. 1.
- link vega_1u_head_l2: geometry collision mesh filename=meshes/vega_1u_head_l2_collisions_head_l2_mesh.obj scale=1. 1. 1.; visual mesh filename=meshes/vega_1u_head_l2_collisions_head_l2_mesh.obj scale=1. 1. 1.
- link vega_1u_head_l3: geometry collision mesh filename=meshes/head_l3_0_mesh.obj scale=1. 1. 1.; collision mesh filename=meshes/head_l3_1_mesh.obj scale=1. 1. 1.
- link vega_1u_lift_link: geometry collision mesh filename=meshes/vega_1u_lift_link_collisions_lift_link_mesh.obj scale=1. 1. 1.; visual mesh filename=meshes/vega_1u_lift_link_collisions_lift_link_mesh.obj scale=1. 1. 1.

Commit message: wip - freeze anchoring function for greater workspace accessibility during teleop

File: robot/vega_1u_gripper.urdf (robot description, URDF)
Before this commit: robot vega_1u_gripper, 35 links, 34 joints
Joints:
- joint L_gripper_joint: limit lower=0. upper=0.6649704 effort=10000000. velocity=2.0 -> lower=0. upper=0.6649704 effort=3. velocity=2.0
- joint R_gripper_joint: limit lower=0. upper=0.6649704 effort=10000000. velocity=2.0 -> lower=0. upper=0.6649704 effort=3. velocity=2.0
